File: drivers_moteurs.kicad_sch (KiCad schematic)
At the start: 21 parts

Commit message: placement des empreintes début
Parts:
- removed MOT1, MOT2, MOT3: Conn_02x04_Row_Letter_Last, Connector_PinHeader_2.54mm:PinHeader_1x04_P2.54mm_Horizontal, symbol Connector_Generic:Conn_02x04_Row_Letter_Last
- added MOT1, MOT3: Conn_02x04_Top_Bottom, Connector_PinHeader_2.54mm:PinHeader_2x04_P2.54mm_Horizontal, symbol Connector_Generic:Conn_02x04_Top_Bottom
- added MOT2: Connector_PinHeader_2.54mm:PinHeader_2x04_P2.54mm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, symbol Connector_Generic:Conn_02x04_Top_Bottom
Connections:
- net GND: now also MOT1.5 (Pin_5), MOT1.6 (Pin_6), MOT1.7 (Pin_7), MOT1.8 (Pin_8), MOT2.5 (Pin_5), MOT2.6 (Pin_6), MOT2.7 (Pin_7), MOT2.8 (Pin_8), MOT3.5 (Pin_5), MOT3.6 (Pin_6), MOT3.7 (Pin_7), MOT3.8 (Pin_8)
- net at DR2.6 (OA1): now also MOT2.1 (Pin_1)
- net at DR2.5 (OA2): now also MOT2.2 (Pin_2)
- net at DR2.4 (OB2): now also MOT2.3 (Pin_3)
- net at DR2.3 (OB1): now also MOT2.4 (Pin_4)
- net at DR3.6 (OA1): now also MOT3.1 (Pin_1)
- net at DR3.5 (OA2): now also MOT3.2 (Pin_2)
- net at DR3.4 (OB2): now also MOT3.3 (Pin_3)
- net at DR3.3 (OB1): now also MOT3.4 (Pin_4)
- net at DR1.3 (OB1): now also MOT1.4 (Pin_4)
- net at DR1.4 (OB2): now also MOT1.3 (Pin_3)
- net at DR1.5 (OA2): now also MOT1.2 (Pin_2)
- net at DR1.6 (OA1): now also MOT1.1 (Pin_1)

Commit message: tout connecté
Parts:
- removed MOT1, MOT3: Conn_02x04_Top_Bottom, Connector_PinHeader_2.54mm:PinHeader_2x04_P2.54mm_Horizontal, symbol Connector_Generic:Conn_02x04_Top_Bottom
- removed MOT2: Connector_PinHeader_2.54mm:PinHeader_2x04_P2.54mm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, symbol Connector_Generic:Conn_02x04_Top_Bottom
- added MOT1, MOT2, MOT3: Conn_02x04_Odd_Even, Connector_PinHeader_2.54mm:PinHeader_2x04_P2.54mm_Horizontal, symbol Connector_Generic:Conn_02x04_Odd_Even
Connections:
- net GND: now also MOT1.2 (Pin_2), MOT1.4 (Pin_4), MOT1.6 (Pin_6), MOT1.8 (Pin_8), MOT2.2 (Pin_2), MOT2.4 (Pin_4), MOT2.6 (Pin_6), MOT2.8 (Pin_8), MOT3.2 (Pin_2), MOT3.4 (Pin_4), MOT3.6 (Pin_6), MOT3.8 (Pin_8)
- net at DR1.6 (OA1): now also MOT1.1 (Pin_1)
- net at DR1.5 (OA2): now also MOT1.3 (Pin_3)
- net at DR1.4 (OB2): now also MOT1.5 (Pin_5)
- net at DR1.3 (OB1): now also MOT1.7 (Pin_7)
- net at DR2.6 (OA1): now also MOT2.1 (Pin_1)
- net at DR2.5 (OA2): now also MOT2.3 (Pin_3)
- net at DR2.4 (OB2): now also MOT2.5 (Pin_5)
- net at DR2.3 (OB1): now also MOT2.7 (Pin_7)
- net at DR3.6 (OA1): now also MOT3.1 (Pin_1)
- net at DR3.5 (OA2): now also MOT3.3 (Pin_3)
- net at DR3.4 (OB2): now also MOT3.5 (Pin_5)
- net at DR3.3 (OB1): now also MOT3.7 (Pin_7)
