File: alimentation.kicad_sch (KiCad schematic)
At the start: 15 parts, among them J3 Conn_01x02, J4 Conn_01x02, J5 Conn_01x02

Commit message: placement des empreintes début
Parts:
- removed ALM1, ALM2, ALM3: Conn_01x02, Connector_AMASS:AMASS_XT30PW-F_1x02_P2.50mm_Horizontal, symbol Connector_Generic:Conn_01x02
- added ALM0: Conn_02x03_Odd_Even, Connector_Molex:Molex_Mini-Fit_Jr_5569-06A2_2x03_P4.20mm_Horizontal, symbol Connector_Generic:Conn_02x03_Odd_Even
- J3, J4, J5: footprint Connector_PinHeader_2.54mm:PinHeader_1x02_P2.54mm_Vertical -> Connector_JST:JST_XH_B2B-XH-A_1x02_P2.50mm_Vertical
Connections:
- net +BATT: now also F1.2; no longer F1.1
- net GND: now also ALM0.1 (Pin_1), ALM0.2 (Pin_2)
- net at F2.2: now also ALM0.4 (Pin_4)
- net at F3.2: now also ALM0.6 (Pin_6)
- new net: ALM0.3 (Pin_3), ALM0.5 (Pin_5), F1.1
Other:
- note added: "Branchements d'alimentation"
- note removed: "Branchements d'alimentation Vbatt, V0, 5V"
- moved on the sheet: C1, C3, F2, F3, J3, J4, J5, JP12, JP13, JP14

Commit message: tout connecté
Parts:
- J3, J4, J5: footprint Connector_JST:JST_XH_B2B-XH-A_1x02_P2.50mm_Vertical -> Connector_JST:JST_XH_S2B-XH-A_1x02_P2.50mm_Horizontal
Connections:
- net VBatt_in: now reaches ALM0.3 (Pin_3), ALM0.5 (Pin_5), F1.1
- net 5V_in: now reaches ALM0.4 (Pin_4)
- net 5V_in: now also F3.2; no longer F2.2
- net V0_in: now reaches ALM0.6 (Pin_6)
- net V0_in: now also F2.2; no longer F3.2
Other:
- moved on the sheet: C2, C3, F2, F3

Commit message: v2 finalisé
Parts:
- removed F1, F2, F3: Fuse, Fuse:Fuse_1206_3216Metric_Pad1.42x1.75mm_HandSolder, symbol Device:Fuse
- renumbered J3 to J1, J5 to J2, J4 to J3
Connections:
- net 5V_in is gone; now on net +5V: ALM0.4 (Pin_4)
- net V0_in is gone; now on net +V0: ALM0.6 (Pin_6)
- net VBatt_in is gone; now on net +BATT: ALM0.3 (Pin_3), ALM0.5 (Pin_5)
Other:
- moved on the sheet: J2, J3

Commit message: paufinement
Parts:
- C3: footprint Capacitor_SMD:CP_Elec_6.3x5.8 -> Capacitor_SMD:CP_Elec_6.3x7.7
Changed lines of the file:
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@@
 			)
 		)
-		(property "Footprint" "Capacitor_SMD:CP_Elec_6.3x5.8"
+		(property "Footprint" "Capacitor_SMD:CP_Elec_6.3x7.7"
 			(at 102.87 44.7548 0)
 			(effects
